File: a44key-pcb.kicad_pcb (KiCad board)
At the start: 2 copper layers, 116.6 x 105.5 mm, 68 parts, among them J1 AudioJack3, J2 Conn_01x04_Female, J3 Conn_01x04_Female, J4 Conn_01x04_Female, SW1 SW_Push, U1 ATmega32U4-AU, Y1 16MHz

Commit message: PCB
Parts:
- moved D21 2.25 mm to (138.2, 90.3)
- moved D18 1.89 mm to (135.6, 90.3)
- moved D22 1.85 mm to (138.4, 109.1)
- moved SW1 1.55 mm to (88.6, 124.5)
- moved D19 1.48 mm to (135.9, 109.1)
- moved D13 1.44 mm to (133.1, 70.7)
- moved D2 1.42 mm to (128.0, 90.3)
- moved D14 1.37 mm to (133.1, 90.3)
- moved R5 1.36 mm to (116.6, 119.6), turned to 90 degrees
- moved D20 1.35 mm to (138.2, 70.7)
- moved D17 1.35 mm to (135.6, 70.7)
- moved D10 1.30 mm to (130.6, 90.3)
- moved D5 1.09 mm to (128.0, 70.7)
- moved D6 1.05 mm to (125.5, 90.3)
- moved D15 1.05 mm to (133.3, 109.1)
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Routing:
- net COL1: track 137.1 -> 282.8 mm, vias 0 -> 3
- net COL0: track 133.4 -> 277.4 mm, vias 0 -> 3
- net ROW0: track 0.00 -> 94.1 mm, vias 0 -> 2
- net ROW1: track 0.00 -> 81.0 mm, vias 0 -> 5
- net TH34: track 0.00 -> 76.3 mm
- net TH35: track 2.82 -> 62.7 mm
- net COL2: track 185.7 -> 244.9 mm
- net ROW2: track 0.00 -> 57.5 mm, vias 0 -> 2
- net Net-(D20-Pad2): track 4.24 -> 57.7 mm
- net Net-(D22-Pad2): track 4.24 -> 57.1 mm
- net Net-(D21-Pad2): track 4.24 -> 56.4 mm
- net ROW3: track 0.00 -> 50.7 mm, vias 0 -> 2
- net Net-(D3-Pad2): track 4.24 -> 40.5 mm
- net Net-(D2-Pad2): track 4.24 -> 40.4 mm
- net Net-(D17-Pad2): track 4.24 -> 39.3 mm
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Other:
- board size 116.6 x 105.5 mm -> 116.7 x 103.9 mm

Commit message: PCB
Parts:
- added Right-Left1: JP1, Jumper:SolderJumper-3_P1.3mm_Open_Pad1.0x1.5mm, B.Cu at (94.0, 133.6)
- J2: moved to F.Cu
- moved D12 3.30 mm to (134.9, 128.1)
- moved D4 3.30 mm to (132.3, 128.1)
- moved D8 3.30 mm to (129.8, 128.1)
- moved D16 3.30 mm to (137.4, 128.1)
- moved R4 1.41 mm to (97.8, 133.1), turned to 90 degrees
- turned J2 to 285 degrees
Connections:
- R4 pad 1: GND -> Net-(R4-Pad1)
Routing:
- net TH34: track 76.3 -> 80.6 mm
- net TH35: track 62.7 -> 66.9 mm
- net ROW3: track 50.7 -> 54.7 mm
- net Net-(R4-Pad1): track 0.00 -> 4.00 mm
- net VCC: track 147.4 -> 150.8 mm
- net Net-(D12-Pad2): track 26.2 -> 24.4 mm
- net Net-(D16-Pad2): track 19.9 -> 19.0 mm
- net COL3: track 189.8 -> 188.9 mm
