File: a44key-pcb-left-hand.kicad_pcb (KiCad board)
At the start: 2 copper layers, 116.7 x 103.9 mm, 69 parts, among them J1 AudioJack3, J2 Conn_01x04_Female, J3 Conn_01x04_Female, J4 Conn_01x04_Female, SW1 SW_Push, U1 ATmega32U4-AU, Y1 16MHz

Commit message: Added parameters for the modifier to work nicelyDD
Parts:
- SW1: moved to F.Cu
- moved Right-Left1 26.6 mm to (155.7, 114.8), turned to 90 degrees
- moved R4 2.03 mm to (179.8, 110.5), turned to 180 degrees
- moved R5 0.30 mm to (161.0, 122.0)
Connections:
- R4 pad 1: Net-(R4-Pad1) -> GND
- R5 pad 1: GND -> Net-(R5-Pad1)
- Right-Left1 pad 2: Net-(R4-Pad1) -> Net-(R5-Pad1)
Routing:
- net Net-(R5-Pad1): track 0.00 -> 11.4 mm
- net VCC: track 136.1 -> 144.2 mm
- net Net-(R3-Pad2): track 24.5 -> 30.2 mm, vias 2 -> 3
- net ROW1: track 94.5 -> 98.8 mm
- net Net-(R1-Pad1): track 112.4 -> 116.5 mm
- net Net-(R2-Pad1): track 117.1 -> 121.0 mm
- net Net-(R4-Pad1): track 3.61 -> 0.00 mm
- net GND: track 176.1 -> 178.8 mm, vias 4 -> 5
- net COL5: track 188.3 -> 186.6 mm
- net Net-(R4-Pad2): track 3.15 -> 1.82 mm
- net COL0: track 260.3 -> 259.2 mm
- net COL1: track 233.0 -> 232.5 mm
